File: Eagle Files/display.brd (EAGLE design)
At the start: 38.4 x 51.4 mm, 14 parts, among them CN1 Charger, IC1 ATMEGA 328P-PU

Commit message: fixed a typo
Parts:
- JP4: value Ananlog IO -> Analog IO
Changed lines of the file:
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@@
 </element>
 <element name="C1" library="resistor" package="C050-025X075" value="100n" x="24.13" y="33.02" smashed="yes" rot="R180">
-<attribute name="NAME" x="23.114" y="32.004" size="1.27" layer="25" ratio="10" rot="R180"/>
-<attribute name="VALUE" x="27.559" y="32.004" size="1.27" layer="27" ratio="10" rot="R180"/>
+<attribute name="NAME" x="22.479" y="31.369" size="1.27" layer="25" ratio="10" rot="R180"/>
+<attribute name="VALUE" x="28.194" y="31.369" size="1.27" layer="27" ratio="10" rot="R180"/>
 </element>
 <element name="JP2" library="pinhead" package="1X07" value="Display" x="19.05" y="46.355" smashed="yes">
@@
 <attribute name="VALUE" x="14.605" y="15.875" size="1.27" layer="27"/>
 </element>
-<element name="JP4" library="adafruit" package="1X06-CLEAN" value="Ananlog IO" x="28.575" y="18.415" smashed="yes">
+<element name="JP4" library="adafruit" package="1X06-CLEAN" value="Analog IO" x="28.575" y="18.415" smashed="yes">
 <attribute name="NAME" x="22.7838" y="18.9738" size="1.27" layer="25" ratio="10"/>
 <attribute name="VALUE" x="21.59" y="15.875" size="1.27" layer="27"/>
